Commit message: Updated workspace for hydro

File: src/mag_simulation/mag_description/urdf/sensors/hokuyo_laser.xacro (robot description, xacro)
@@ -9,5 +9,5 @@
     <link name="hokuyo_link" type="laser">
 		  <visual>
-		  	<origin xyz="0 0 0.08" />
+		  	<origin xyz="0 0 0.07" />
 		    <geometry>
 					<mesh filename="package://mag_description/meshes/hokuyo_laser.dae"/>
@@ -15,5 +15,5 @@
 		  </visual>
 		  <collision>
-		  	<origin xyz="0 0 0.08" />
+		  	<origin xyz="0 0 0.7" />
 		    <geometry>
 		      <box size="0.05 0.05 0.1" />
@@ -21,5 +21,5 @@
 		  </collision>
       <inertial>
-		  	<origin xyz="0 0 0.08" />
+		  	<origin xyz="0 0 0.07" />
         <mass value="0.1" />
         <inertia ixx="0.0001" ixy="0" ixz="0" iyy="0.0001" iyz="0" izz="0.0001" />
