Commit message: Fixed bugs in URDF model and window nav

File: src/mag_simulation/mag_description/urdf/parts/caster.xacro (robot description, xacro)
@@ -19,5 +19,5 @@
 			<inertial>
 				<origin rpy="${PI/2} 0 ${PI/2}"/>
-				<mass value="10"/>
+				<mass value="5"/>
 				<inertia ixx="0.4" ixy="0.0" ixz="0.0" iyy="0.4" iyz="0.0" izz="0.2"/>
 			</inertial>

File: src/mag_simulation/mag_description/urdf/parts/chassis.xacro (robot description, xacro)
@@ -22,5 +22,5 @@
 			<inertial>
 				<origin xyz="0 0 ${height/2}"/>
-				<mass value="10"/>
+				<mass value="20"/>
 				<inertia ixx="0.4" ixy="0.0" ixz="0.0" iyy="0.4" iyz="0.0" izz="0.2"/>
 			</inertial>

File: src/mag_simulation/mag_description/urdf/parts/wheel.xacro (robot description, xacro)
@@ -27,5 +27,5 @@
 		  <parent link="base_link"/>
 		  <child link="${name}"/>
-		  <axis xyz="1 0 0"/>
+		  <axis xyz="-1 0 0"/>
 		  <insert_block name="origin" />
 		</joint>
