Commit message: Fixed some topics and added Sensors urdf and meshes

File: src/mag_simulation/mag_description/urdf/magabot.xacro (robot description, xacro)
@@ -11,7 +11,12 @@
   <xacro:property name="centerWidth" value="0.01"/> <!-- Width of non-motorized wheel -->
   <xacro:property name="axel_offset" value="0.05"/> <!-- Space btw top of beam and the each joint -->
-  <!-- Import Gazebo customization elements -->
+  <!-- Sensor TFs -->
+  <xacro:macro name="hokuyo_tf"> <origin xyz="0 0.0305 0.0871" rpy="0 0 0"/> </xacro:macro>
+	<xacro:macro name="wiimote_tf"> <origin xyz="0 -0.0721 0.072" rpy="0 0 0"/> </xacro:macro>
+  <!-- Import Gazebo elements -->
   <xacro:include filename="$(find mag_description)/urdf/magabot.gazebo" />
-  <!-- Import Rviz colors -->
+  <!-- Import Sensors -->
+  <xacro:include filename="$(find mag_description)/urdf/sensors/hokuyo_laser.xacro" />
+  <!-- Import Materials -->
   <xacro:include filename="$(find mag_description)/urdf/materials.xacro" />
   <!-- Macro for motorized wheels -->
@@ -39,5 +44,5 @@
 		  <parent link="base_link"/>
 		  <child link="${name}"/>
-		  <axis xyz="0 1 0"/>
+		  <axis xyz="1 0 0"/>
 		  <origin xyz="${reflect*.15} .1 0" rpy="0 0 0"/>
 		</joint>
@@ -50,5 +55,5 @@
   			<box size="${width} ${length} ${height}"/>
   		</geometry>
-  		<material name="orange"/>-
+  		<material name="orange"/>
   	</visual>
   	<collision>
@@ -89,5 +94,5 @@
     <parent link="base_link"/>
     <child link="centerwheel"/>
-    <axis xyz="0 0 1"/>
+    <axis xyz="1 0 0"/>
     <origin xyz="0 -.1 0" rpy="0 0 0"/>
   </joint>
@@ -109,3 +114,7 @@
     </actuator>
   </transmission>
+  <!-- ....... SENSORS ....... -->
+  <xacro:hokuyo_laser parent="base_link">
+  	<xacro:hokuyo_tf/>
+  </xacro:hokuyo_laser>
 </robot>

Commit message: Fixed several URDFs

File: src/mag_simulation/mag_description/urdf/magabot.xacro (robot description, xacro)
@@ -18,4 +18,5 @@
   <!-- Import Sensors -->
   <xacro:include filename="$(find mag_description)/urdf/sensors/hokuyo_laser.xacro" />
+  <xacro:include filename="$(find mag_description)/urdf/sensors/microstrain.xacro" />
   <!-- Import Materials -->
   <xacro:include filename="$(find mag_description)/urdf/materials.xacro" />
@@ -63,4 +64,7 @@
   		</geometry>
   	</collision>
+  </link>
+  <!-- Dummy link to associate inertia with base_link, to avoid errors in simulation -->
+  <link name="base_inertia">
 		<inertial>
   		<origin xyz="0 0 0.1" rpy="0 0 0"/>
@@ -68,5 +72,5 @@
 			<inertia ixx="0.4" ixy="0.0" ixz="0.0" iyy="0.4" iyz="0.0" izz="0.2"/>
 		</inertial>
-  </link>
+	</link>
   <xacro:wheel name="leftwheel" reflect="1"/>
   <xacro:wheel name="rightwheel" reflect="-1"/>
@@ -91,4 +95,10 @@
   </link>
   <!-- ........... JOINTS ........... -->
+  <joint name="base_inertia_joint" type="fixed">
+  	<parent link="base_link"/>
+  	<child link="base_inertia"/>
+  	<axis xyz="1 0 0"/>
+  	<origin xyz="0 0 0" rpy="0 0 0"/>
+  </joint>
   <joint name="base_centerwheel" type="continuous">
     <parent link="base_link"/>
@@ -98,5 +108,5 @@
   </joint>
   <!-- ........... TRANSMISSIONS ........... -->
-  <transmission name="leftTrans">
+  <transmission name="leftTransmission">
     <type>transmission_interface/SimpleTransmission</type>
     <joint name="base_leftwheel"/>
@@ -106,5 +116,5 @@
     </actuator>
   </transmission>
-  <transmission name="rightTrans">
+  <transmission name="rightTransmission">
     <type>transmission_interface/SimpleTransmission</type>
     <joint name="base_rightwheel"/>
@@ -115,6 +125,9 @@
   </transmission>
   <!-- ....... SENSORS ....... -->
-  <xacro:hokuyo_laser parent="base_link">
+  <xacro:hokuyo_laser parent="base_link" topic="laser_scan">
   	<xacro:hokuyo_tf/>
   </xacro:hokuyo_laser>
+  <xacro:microstrain parent="base_link" topic="odom_combined">
+  	<xacro:wiimote_tf/>
+  </xacro:microstrain>
 </robot>

File: src/mag_simulation/mag_description/urdf/sensors/hokuyo_laser.gazebo.xacro (robot description, xacro)
@@ -1,5 +1,5 @@
 <?xml version="1.0"?>
 <robot xmlns:xacro="http://ros.org/wiki/xacro">
-	<xacro:macro name="hokuyo_laser_gazebo">
+	<xacro:macro name="hokuyo_laser_gazebo" params="topic">
 		<!-- hokuyo sensor -->
 		<gazebo reference="hokuyo_link">
@@ -33,5 +33,5 @@
 		    </ray>
 		    <plugin name="gazebo_ros_head_hokuyo_controller" filename="libgazebo_ros_gpu_laser.so">
-		      <topicName>laser_scan</topicName>
+		      <topicName>${topic}</topicName>
 		      <frameName>hokuyo_link</frameName>
 		    </plugin>

File: src/mag_simulation/mag_description/urdf/sensors/hokuyo_laser.xacro (robot description, xacro)
@@ -5,11 +5,11 @@
        xmlns:xacro="http://ros.org/wiki/xacro">
 	<!-- Inlude Gazebo element -->
-  <xacro:include filename="$(find mag_description)/urdf/sensors/hokuyo_laser.gazebo.xacro" />
-  <xacro:macro name="hokuyo_laser" params="parent *origin">
+  <include filename="$(find mag_description)/urdf/sensors/hokuyo_laser.gazebo.xacro" />
+  <xacro:macro name="hokuyo_laser" params="parent *origin topic">
     <link name="hokuyo_link" type="laser">
 		  <visual>
 		    <insert_block name="origin" />
 		    <geometry>
-		      <box size="0.05 0.05 0.1" />
+					<mesh filename="package://mag_description/meshes/hokuyo_laser.dae"/>
 		    </geometry>
 		  </visual>
@@ -33,5 +33,5 @@
     </joint>
     <!-- Gazebo elements -->
-    <xacro:hokuyo_laser_gazebo/>
+    <xacro:hokuyo_laser_gazebo topic="${topic}"/>
   </xacro:macro>
 </robot>

File: src/mag_simulation/mag_description/urdf/sensors/microstrain.gazebo.xacro (robot description, xacro)
@@ -1,20 +1,19 @@
 <?xml version="1.0"?>
-<robot xmlns:sensor="http://playerstage.sourceforge.net/gazebo/xmlschema/#sensor"
-				xmlns:controller="http://playerstage.sourceforge.net/gazebo/xmlschema/#controller"
-				xmlns:interface="http://playerstage.sourceforge.net/gazebo/xmlschema/#interface"
-				xmlns:xacro="http://ros.org/wiki/xacro">
-	<xacro:macro name="microstrain_gazebo" params="name imu_topic update_rate stdev">
-		<gazebo>
-			<controller:gazebo_ros_imu name="imu_controller" plugin="libgazebo_ros_imu.so">
-				<alwaysOn>true</alwaysOn>
-				<updateRate>80</updateRate>
-				<bodyName>microstrain_link</bodyName>
-				<topicName>imu_data</topicName>
-				<gaussianNoise>0.0001</gaussianNoise>
-				<xyzOffsets>0 0 0</xyzOffsets>
-				<rpyOffsets>0 0 0</rpyOffsets>
-				<interface:position name="imu_position"/>
-			</controller:gazebo_ros_imu>
-		</gazebo>
-	</xacro:macro>
+<robot xmlns:controller="http://playerstage.sourceforge.net/gazebo/xmlschema/#controller"
+       xmlns:interface="http://playerstage.sourceforge.net/gazebo/xmlschema/#interface"
+       xmlns:xacro="http://ros.org/wiki/xacro">
+  <xacro:macro name="microstrain_gazebo" params="topic">
+    <gazebo>
+      <plugin name="imu_controller" filename="libgazebo_ros_imu.so">
+        <alwaysOn>true</alwaysOn>
+        <updateRate>80</updateRate>
+        <bodyName>microstrain_link</bodyName>
+        <topicName>${topic}</topicName>
+        <serviceName>/default_imu</serviceName>
+        <gaussianNoise>0.0000000289</gaussianNoise> <!-- 0.00017 * 0.00017 -->
+        <xyzOffset>0 0 0</xyzOffset>
+        <rpyOffset>0 -180.0 0</rpyOffset>
+      </plugin>
+    </gazebo>
+  </xacro:macro>
 </robot>

File: src/mag_simulation/mag_description/urdf/sensors/microstrain.xacro (robot description, xacro)
@@ -6,5 +6,5 @@
 	<!-- Include Gazebo element -->
 	<include filename="$(find mag_description)/urdf/sensors/microstrain.gazebo.xacro" />
-	<xacro:macro name="microstrain" params="parent *origin">
+	<xacro:macro name="microstrain" params="parent *origin topic">
 		<link name="microstrain_link">
 		  <visual>
@@ -21,7 +21,7 @@
 		  </collision>
 			<inertial>
-				<mass value="0.001" />
+				<mass value="0.01" />
 				<origin xyz="0 0 0" rpy="0 0 0" />
-				<inertia ixx="0.0001" ixy="0" ixz="0" iyy="0.000001" iyz="0" izz="0.0001" />
+				<inertia ixx="0.0001" ixy="0" ixz="0" iyy="0.0001" iyz="0" izz="0.0001" />
 			</inertial>
 		</link>
@@ -33,5 +33,5 @@
 		</joint>
 		<!-- Gazebo element -->
-		<xacro:microstrain_gazebo/>
+		<xacro:microstrain_gazebo topic="${topic}"/>
 	</xacro:macro>
 </robot>

File: src/mag_simulation/mag_description/urdf/sensors/xtion.gazebo.xacro (robot description, xacro)
@@ -4,8 +4,7 @@
 				xmlns:interface="http://playerstage.sourceforge.net/gazebo/xmlschema/#interface"
 				xmlns:xacro="http://ros.org/wiki/xacro">
-	<xacro:macro name="xtion_gazebo" params="name parent *origin">
-		<!-- ASUS Xtion PRO camera for simulation -->
-		<gazebo reference="${name}_depth_frame">
-			<sensor:camera name="${name}">
+	<xacro:macro name="xtion_gazebo" params="topic">
+		<gazebo reference="xtion_depth_frame">
+			<sensor:camera name="xtion">
 				<imageFormat>R8G8B8</imageFormat>
 				<imageSize>640 480</imageSize>
@@ -15,18 +14,18 @@
 				<updateRate>20</updateRate>
 				<baseline>0.1</baseline>
-				<controller:gazebo_ros_openni_kinect name="${name}_camera_controller" plugin="libgazebo_ros_openni_kinect.so">
-				<alwaysOn>true</alwaysOn>
-				<updateRate>20</updateRate>
-				<imageTopicName>${name}/rgb/image_raw</imageTopicName>
-				<cameraInfoTopicName>${name}/rgb/camera_info</cameraInfoTopicName>
-				<depthImageTopicName>${name}/depth/image_raw</depthImageTopicName>
-				<depthImageCameraInfoTopicName>${name}/depth/camera_info</depthImageCameraInfoTopicName>
-				<pointCloudTopicName>${name}/depth/points</pointCloudTopicName>
-				<frameName>${name}_depth_optical_frame</frameName>
-				<distortion_k1>0.0</distortion_k1>
-				<distortion_k2>0.0</distortion_k2>
-				<distortion_k3>0.0</distortion_k3>
-				<distortion_t1>0.0</distortion_t1>
-				<distortion_t2>0.0</distortion_t2>
+				<controller:gazebo_ros_openni_kinect name="xtion_camera_controller" plugin="libgazebo_ros_openni_kinect.so">
+					<alwaysOn>true</alwaysOn>
+					<updateRate>20</updateRate>
+					<imageTopicName>xtion/rgb/image_raw</imageTopicName>
+					<cameraInfoTopicName>xtion/rgb/camera_info</cameraInfoTopicName>
+					<depthImageTopicName>${topic}</depthImageTopicName>
+					<depthImageCameraInfoTopicName>xtion/depth/camera_info</depthImageCameraInfoTopicName>
+					<pointCloudTopicName>xtion/depth/points</pointCloudTopicName>
+					<frameName>xtion_frame</frameName>
+					<distortion_k1>0.0</distortion_k1>
+					<distortion_k2>0.0</distortion_k2>
+					<distortion_k3>0.0</distortion_k3>
+					<distortion_t1>0.0</distortion_t1>
+					<distortion_t2>0.0</distortion_t2>
 				</controller:gazebo_ros_openni_kinect>
 			</sensor:camera>

File: src/mag_simulation/mag_description/urdf/sensors/xtion.xacro (robot description, xacro)
@@ -7,5 +7,5 @@
 	<include filename="$(find mag_description)/urdf/sensors/xtion.gazebo.xacro" />
 	<property name="PI" value="3.1415926" />
-	<xacro:macro name="xtion" params="parent *origin">
+	<xacro:macro name="xtion" params="parent *origin topic">
 		<joint name="xtion_joint" type="fixed">
 			<insert_block name="origin" />
@@ -57,5 +57,5 @@
 		<link name="xtion_rgb_optical_frame"/>
 		<!-- Gazebo element -->
-		<xacro:microstrain_gazebo/>
+		<xacro:microstrain_gazebo topic="${topic}"/>
 	</xacro:macro>
 </robot>

Commit message: Separated urdf description and fixed some bugs in urdf

File: src/mag_simulation/mag_description/urdf/magabot.xacro (robot description, xacro)
@@ -3,130 +3,49 @@
   <!-- Constants with robot dimensions -->
   <xacro:property name="PI" value="3.14159"/>
-  <xacro:property name="width" value="0.384602"/> <!-- Width of the base chassis -->
-  <xacro:property name="length" value="0.451048"/> <!-- Length of the base chassis -->
-  <xacro:property name="height" value="0.10165"/> <!-- Height of the base chassis -->g
-  <xacro:property name="wheelRadius" value="0.0463"/> <!-- Radius of motorized wheels -->
-  <xacro:property name="wheelWidth" value="0.01"/> <!-- Width of motorized wheels -->
-  <xacro:property name="centerRadius" value="0.0463"/> <!-- Radius of non-motorized wheel -->
-  <xacro:property name="centerWidth" value="0.01"/> <!-- Width of non-motorized wheel -->
-  <xacro:property name="axel_offset" value="0.05"/> <!-- Space btw top of beam and the each joint -->
+  <xacro:property name="width" value="0.3846"/> <!-- Width of the base chassis -->
+  <xacro:property name="length" value="0.451"/> <!-- Length of the base chassis -->
+  <xacro:property name="height" value="0.06826"/> <!-- Height of the base chassis -->
+  <xacro:property name="wheelRadius" value="0.045"/> <!-- Radius of motorized wheels -->
+  <xacro:property name="wheelWidth" value="0.0108"/> <!-- Width of motorized wheels -->
+  <xacro:property name="wheelSep" value="0.345"/> <!-- Distance between wheels, for Differential Drive -->
+  <xacro:property name="casterRadius" value="0.0225"/> <!-- Radius of non-motorized wheel -->
+  <xacro:property name="casterWidth" value="0.020"/> <!-- Width of non-motorized wheel -->
+  <!-- Magabot TFs -->
+  <xacro:macro name="footprint_tf"> <origin xyz="0 0 0.0307" rpy="0 0 0"/> </xacro:macro>
+  <xacro:macro name="wheel_tf" params="reflect"> <origin xyz="${reflect*.1725} .0455 0.0143" rpy="0 0 0"/> </xacro:macro>
+  <xacro:macro name="caster_tf"> <origin xyz="0 -0.169 -0.0092" rpy="0 0 0"/> </xacro:macro>
   <!-- Sensor TFs -->
-  <xacro:macro name="hokuyo_tf"> <origin xyz="0 0.0305 0.0871" rpy="0 0 0"/> </xacro:macro>
-	<xacro:macro name="wiimote_tf"> <origin xyz="0 -0.0721 0.072" rpy="0 0 0"/> </xacro:macro>
-  <!-- Import Gazebo elements -->
+  <xacro:macro name="hokuyo_tf"> <origin xyz="0 0.0305 ${height}" rpy="0 0 0"/> </xacro:macro>
+	<xacro:macro name="wiimote_tf"> <origin xyz="0 -0.0721 ${height}" rpy="0 0 0"/> </xacro:macro>
+  <!-- Import Magabot Gazebo elements -->
   <xacro:include filename="$(find mag_description)/urdf/magabot.gazebo" />
+  <xacro:plugins_gazebo topic="odom_combined" wheelSep="${wheelSep}" wheelRad="${wheelRadius}"/> <xacro:magabot_gazebo/>
+	<!-- Import Parts -->
+	<xacro:include filename="$(find mag_description)/urdf/parts/chassis.xacro" />
+	<xacro:include filename="$(find mag_description)/urdf/parts/wheel.xacro" />
+	<xacro:include filename="$(find mag_description)/urdf/parts/caster.xacro" />
   <!-- Import Sensors -->
   <xacro:include filename="$(find mag_description)/urdf/sensors/hokuyo_laser.xacro" />
   <xacro:include filename="$(find mag_description)/urdf/sensors/microstrain.xacro" />
   <!-- Import Materials -->
-  <xacro:include filename="$(find mag_description)/urdf/materials.xacro" />
-  <!-- Macro for motorized wheels -->
-  <xacro:macro name="wheel" params="name reflect">
-  	<link name="${name}">
-			<visual>
-				<origin xyz="0 0 0" rpy="${PI/2} 0 ${PI/2}"/>
-				<geometry>
-					<cylinder length="${wheelWidth}" radius="${wheelRadius}"/>
-				</geometry>
-				<material name="blue"/>
-			</visual>
-			<collision>
-				<origin xyz="0 0 0" rpy="${PI/2} 0 ${PI/2}"/>
-				<geometry>
-					<cylinder length="${wheelWidth}" radius="${wheelRadius}"/>
-				</geometry>
-			</collision>
-			<inertial>
-				<mass value="10"/>
-				<inertia ixx="0.4" ixy="0.0" ixz="0.0" iyy="0.4" iyz="0.0" izz="0.2"/>
-			</inertial>
-		</link>
-		<joint name="base_${name}" type="continuous">
-		  <parent link="base_link"/>
-		  <child link="${name}"/>
-		  <axis xyz="1 0 0"/>
-		  <origin xyz="${reflect*.15} .1 0" rpy="0 0 0"/>
-		</joint>
-	</xacro:macro>
-  <!-- ........... LINKS ........... -->
-  <link name="base_link">
-  	<visual>
-  		<origin xyz="0 0 0.1" rpy="0 0 0"/>
-  		<geometry>
-  			<box size="${width} ${length} ${height}"/>
-  		</geometry>
-  		<material name="orange"/>
-  	</visual>
-  	<collision>
-  		<origin xyz="0 0 0.1" rpy="0 0 0"/>
-  		<geometry>
-  			<box size="${length} ${width} ${height}"/>
-  		</geometry>
-  	</collision>
-  </link>
-  <!-- Dummy link to associate inertia with base_link, to avoid errors in simulation -->
-  <link name="base_inertia">
-		<inertial>
-  		<origin xyz="0 0 0.1" rpy="0 0 0"/>
-			<mass value="10"/>
-			<inertia ixx="0.4" ixy="0.0" ixz="0.0" iyy="0.4" iyz="0.0" izz="0.2"/>
-		</inertial>
-	</link>
-  <xacro:wheel name="leftwheel" reflect="1"/>
-  <xacro:wheel name="rightwheel" reflect="-1"/>
-  <link name="centerwheel">
-  	<visual>
-  		<origin xyz="0 0 0" rpy="${PI/2} 0 ${PI/2}"/>
-  		<geometry>
-  			<cylinder length="${centerWidth}" radius="${centerRadius}"/>
-  		</geometry>
-  		<material name="Blue"/>
-  	</visual>
-  	<collision>
-  		<origin xyz="0 0 0" rpy="${PI/2} 0 ${PI/2}"/>
-  		<geometry>
-  			<cylinder length="${centerWidth}" radius="${centerRadius}"/>
-  		</geometry>
-  	</collision>
-		<inertial>
-			<mass value="10"/>
-			<inertia ixx="0.4" ixy="0.0" ixz="0.0" iyy="0.4" iyz="0.0" izz="0.2"/>
-		</inertial>
-  </link>
-  <!-- ........... JOINTS ........... -->
-  <joint name="base_inertia_joint" type="fixed">
-  	<parent link="base_link"/>
-  	<child link="base_inertia"/>
-  	<axis xyz="1 0 0"/>
-  	<origin xyz="0 0 0" rpy="0 0 0"/>
-  </joint>
-  <joint name="base_centerwheel" type="continuous">
-    <parent link="base_link"/>
-    <child link="centerwheel"/>
-    <axis xyz="1 0 0"/>
-    <origin xyz="0 -.1 0" rpy="0 0 0"/>
-  </joint>
-  <!-- ........... TRANSMISSIONS ........... -->
-  <transmission name="leftTransmission">
-    <type>transmission_interface/SimpleTransmission</type>
-    <joint name="base_leftwheel"/>
-    <actuator name="leftMotor">
-      <hardwareInterface>EffortJointInterface</hardwareInterface>
-      <mechanicalReduction>1</mechanicalReduction>
-    </actuator>
-  </transmission>
-  <transmission name="rightTransmission">
-    <type>transmission_interface/SimpleTransmission</type>
-    <joint name="base_rightwheel"/>
-    <actuator name="motorRight">
-      <hardwareInterface>EffortJointInterface</hardwareInterface>
-      <mechanicalReduction>1</mechanicalReduction>
-    </actuator>
-  </transmission>
+  <xacro:include filename="$(find mag_description)/urdf/materials/materials.xacro" />
+  <!-- ........... PARTS ........... -->
+  <xacro:chassis width="${width}" length="${length}" height="${height}">
+  	<xacro:footprint_tf/>
+  </xacro:chassis>
+  <xacro:wheel name="leftwheel" wheelWidth="${wheelWidth}" wheelRadius="${wheelRadius}">
+  	<xacro:wheel_tf reflect="-1" />
+  </xacro:wheel>
+  <xacro:wheel name="rigthwheel" wheelWidth="${wheelWidth}" wheelRadius="${wheelRadius}">
+  	<xacro:wheel_tf reflect="1" />
+  </xacro:wheel>
+  <xacro:caster casterRadius="${casterRadius}" casterWidth="${casterWidth}">
+  	<xacro:caster_tf />
+  </xacro:caster>
   <!-- ....... SENSORS ....... -->
   <xacro:hokuyo_laser parent="base_link" topic="laser_scan">
   	<xacro:hokuyo_tf/>
   </xacro:hokuyo_laser>
-  <xacro:microstrain parent="base_link" topic="odom_combined">
+  <xacro:microstrain parent="base_link" topic="imu_data">
   	<xacro:wiimote_tf/>
   </xacro:microstrain>

File: src/mag_simulation/mag_description/urdf/sensors/microstrain.gazebo.xacro (robot description, xacro)
@@ -13,5 +13,5 @@
         <gaussianNoise>0.0000000289</gaussianNoise> <!-- 0.00017 * 0.00017 -->
         <xyzOffset>0 0 0</xyzOffset>
-        <rpyOffset>0 -180.0 0</rpyOffset>
+        <rpyOffset>0 -180 0</rpyOffset>
       </plugin>
     </gazebo>

File: src/mag_simulation/mag_description/urdf/sensors/microstrain.xacro (robot description, xacro)
@@ -11,5 +11,5 @@
 		    <insert_block name="origin" />
 		    <geometry>
-		      <box size="0.173 0.1585 0.1241" />
+		      <box size="0.0173 0.01585 0.01241" />
 		    </geometry>
 		  </visual>
@@ -17,10 +17,10 @@
 		    <insert_block name="origin" />
 		    <geometry>
-		      <box size="0.173 0.1585 0.1241" />
+		      <box size="0.0173 0.01585 0.01241" />
 		    </geometry>
 		  </collision>
 			<inertial>
+		    <insert_block name="origin" />
 				<mass value="0.01" />
-				<origin xyz="0 0 0" rpy="0 0 0" />
 				<inertia ixx="0.0001" ixy="0" ixz="0" iyy="0.0001" iyz="0" izz="0.0001" />
 			</inertial>
