Commit message: Fixed some URDF errors

File: src/mag_simulation/mag_description/urdf/magabot.xacro (robot description, xacro)
@@ -16,9 +16,8 @@
   <xacro:macro name="caster_tf"> <origin xyz="0 -0.169 -0.0092" rpy="0 0 0"/> </xacro:macro>
   <!-- Sensor TFs -->
-  <xacro:macro name="hokuyo_tf"> <origin xyz="0 0.0305 ${height}" rpy="0 0 0"/> </xacro:macro>
-	<xacro:macro name="wiimote_tf"> <origin xyz="0 -0.0721 ${height}" rpy="0 0 0"/> </xacro:macro>
-  <!-- Import Magabot Gazebo elements -->
+  <xacro:macro name="hokuyo_tf"> <origin xyz="0 0.0305 ${height/2}" rpy="0 0 0"/> </xacro:macro>
+	<xacro:macro name="wiimote_tf"> <origin xyz="0 -0.0721 ${height/2}" rpy="0 0 0"/> </xacro:macro>
+  <!-- Import Gazebo plugins -->
   <xacro:include filename="$(find mag_description)/urdf/magabot.gazebo" />
-  <xacro:plugins_gazebo topic="odom_combined" wheelSep="${wheelSep}" wheelRad="${wheelRadius}"/> <xacro:magabot_gazebo/>
 	<!-- Import Parts -->
 	<xacro:include filename="$(find mag_description)/urdf/parts/chassis.xacro" />
@@ -30,5 +29,5 @@
   <!-- Import Materials -->
   <xacro:include filename="$(find mag_description)/urdf/materials/materials.xacro" />
-  <!-- ........... PARTS ........... -->
+  <!-- ........... MAGABOT PARTS ........... -->
   <xacro:chassis width="${width}" length="${length}" height="${height}">
   	<xacro:footprint_tf/>
@@ -37,5 +36,5 @@
   	<xacro:wheel_tf reflect="-1" />
   </xacro:wheel>
-  <xacro:wheel name="rigthwheel" wheelWidth="${wheelWidth}" wheelRadius="${wheelRadius}">
+  <xacro:wheel name="rightwheel" wheelWidth="${wheelWidth}" wheelRadius="${wheelRadius}">
   	<xacro:wheel_tf reflect="1" />
   </xacro:wheel>
@@ -50,3 +49,5 @@
   	<xacro:wiimote_tf/>
   </xacro:microstrain>
+  <!-- ....... GAZEBO PLUGINS ....... -->
+  <xacro:plugins_gazebo topic="odom_combined" wheelSep="${wheelSep}" wheelRad="${wheelRadius}"/>
 </robot>

File: src/mag_simulation/mag_description/urdf/parts/caster.xacro (robot description, xacro)
@@ -3,5 +3,5 @@
   <xacro:macro name="caster" params="casterWidth casterRadius *origin">
 		<!-- URDF description -->
-		<link name="caster">
+		<link name="caster"> <!-- Caster link -->
 			<visual>
 				<origin rpy="${PI/2} 0 ${PI/2}"/>

File: src/mag_simulation/mag_description/urdf/parts/wheel.xacro (robot description, xacro)
@@ -3,5 +3,5 @@
   <xacro:macro name="wheel" params="name wheelWidth wheelRadius *origin">
 		<!-- URDF description -->
-  	<link name="${name}">
+  	<link name="${name}"> <!-- Motorized wheel link -->
 			<visual>
 				<origin rpy="${PI/2} 0 ${PI/2}"/>

File: src/mag_simulation/mag_description/urdf/sensors/hokuyo_laser.gazebo.xacro (robot description, xacro)
@@ -1,41 +1,36 @@
 <?xml version="1.0"?>
 <robot xmlns:xacro="http://ros.org/wiki/xacro">
-	<xacro:macro name="hokuyo_laser_gazebo" params="topic">
-		<!-- hokuyo sensor -->
-		<gazebo reference="hokuyo_link">
-		  <sensor type="gpu_ray" name="hokuyo_sensor">
-		    <pose>0 0 0 0 0 0</pose>
-		    <visualize>true</visualize>
-		    <update_rate>80</update_rate>
-		    <ray>
-		      <scan>
-		        <horizontal>
-		          <samples>720</samples>
-		          <resolution>1</resolution>
-		          <min_angle>-1.570796</min_angle>
-		          <max_angle>1.570796</max_angle>
-		        </horizontal>
-		      </scan>
-		      <range>
-		        <min>0.10</min>
-		        <max>30.0</max>
-		        <resolution>0.01</resolution>
-		      </range>
-		      <noise>
-		        <type>gaussian</type>
-		        <!-- Noise parameters based on published spec for Hokuyo laser -->
-		        <!--     achieving "+-30mm" accuracy at range < 10m. A mean of 0.0m and -->
-		        <!--     stddev of 0.01m will put 99.7% of samples within 0.03m of the true -->
-		        <!--     reading. -->
-		        <mean>0.0</mean>
-		        <stddev>0.01</stddev>
-		      </noise>
-		    </ray>
-		    <plugin name="gazebo_ros_head_hokuyo_controller" filename="libgazebo_ros_gpu_laser.so">
-		      <topicName>${topic}</topicName>
-		      <frameName>hokuyo_link</frameName>
-		    </plugin>
-		  </sensor>
-		</gazebo>
+  <xacro:macro name="hokuyo_laser_gazebo" params="topic">
+    <gazebo reference="hokuyo_link">
+      <sensor type="ray" name="hokuyo_laser">
+        <pose>0 0 0 0 0 0</pose>
+        <always_on>true</always_on>
+        <visualize>true</visualize>
+        <update_rate>80</update_rate>
+        <ray>
+          <scan>
+            <horizontal>
+              <samples>720</samples>
+              <resolution>1</resolution>
+              <min_angle>-1.570796</min_angle>
+              <max_angle>1.570796</max_angle>
+            </horizontal>
+          </scan>
+          <range>
+            <min>0.1</min>
+            <max>30.0</max>
+            <resolution>0.01</resolution>
+          </range>
+        </ray>
+        <plugin name="gazebo_ros_hokuyo_controller" filename="libgazebo_ros_laser.so">
+          <alwaysOn>true</alwaysOn>
+          <updateRate>80</updateRate>
+          <gaussianNoise>0.005</gaussianNoise>
+          <hokuyoMinIntensity>101</hokuyoMinIntensity>
+          <topicName>${topic}</topicName>
+          <frameName>hokuyo_link</frameName>
+        </plugin>
+      </sensor>
+    </gazebo>
   </xacro:macro>
 </robot>

File: src/mag_simulation/mag_description/urdf/sensors/hokuyo_laser.xacro (robot description, xacro)
@@ -9,5 +9,5 @@
     <link name="hokuyo_link" type="laser">
 		  <visual>
-		    <insert_block name="origin" />
+		  	<origin xyz="0 0 0.08" />
 		    <geometry>
 					<mesh filename="package://mag_description/meshes/hokuyo_laser.dae"/>
@@ -15,5 +15,5 @@
 		  </visual>
 		  <collision>
-		    <insert_block name="origin" />
+		  	<origin xyz="0 0 0.08" />
 		    <geometry>
 		      <box size="0.05 0.05 0.1" />
@@ -21,14 +21,14 @@
 		  </collision>
       <inertial>
-        <mass value="0.01" />
-        <origin xyz="0 0 0" rpy="0 0 0" />
+		  	<origin xyz="0 0 0.08" />
+        <mass value="0.1" />
         <inertia ixx="0.0001" ixy="0" ixz="0" iyy="0.0001" iyz="0" izz="0.0001" />
       </inertial>
     </link>
     <joint name="hokuyo_joint" type="fixed">
+      <parent link="${parent}"/>
+      <child link="hokuyo_link"/>
       <axis xyz="0 1 0" />
       <insert_block name="origin" />
-      <parent link="${parent}"/>
-      <child link="hokuyo_link"/>
     </joint>
     <!-- Gazebo elements -->

Commit message: Fixed sensors in gazebo and tuned the navigation

File: src/mag_simulation/mag_description/urdf/magabot.xacro (robot description, xacro)
@@ -12,9 +12,9 @@
   <xacro:property name="casterWidth" value="0.020"/> <!-- Width of non-motorized wheel -->
   <!-- Magabot TFs -->
-  <xacro:macro name="footprint_tf"> <origin xyz="0 0 0.0307" rpy="0 0 0"/> </xacro:macro>
-  <xacro:macro name="wheel_tf" params="reflect"> <origin xyz="${reflect*.1725} .0455 0.0143" rpy="0 0 0"/> </xacro:macro>
-  <xacro:macro name="caster_tf"> <origin xyz="0 -0.169 -0.0092" rpy="0 0 0"/> </xacro:macro>
+  <xacro:macro name="footprint_tf"> <origin xyz="0 0 ${height/2+0.0307}" rpy="0 0 0"/> </xacro:macro>
+  <xacro:macro name="wheel_tf" params="reflect"> <origin xyz="${reflect*.1725} .0455 ${-height/2+0.0143}" rpy="${PI/2} 0 ${PI/2}"/> </xacro:macro>
+  <xacro:macro name="caster_tf"> <origin xyz="0 -0.169 ${-height/2-0.0092}" rpy="${PI/2} 0 ${PI/2}"/> </xacro:macro>
   <!-- Sensor TFs -->
-  <xacro:macro name="hokuyo_tf"> <origin xyz="0 0.0305 ${height/2}" rpy="0 0 0"/> </xacro:macro>
+  <xacro:macro name="hokuyo_tf"> <origin xyz="0 0.0305 ${height/2+0.035}" rpy="0 0 ${PI/2}"/> </xacro:macro>
 	<xacro:macro name="wiimote_tf"> <origin xyz="0 -0.0721 ${height/2}" rpy="0 0 0"/> </xacro:macro>
   <!-- Import Gazebo plugins -->

File: src/mag_simulation/mag_description/urdf/parts/caster.xacro (robot description, xacro)
@@ -5,5 +5,4 @@
 		<link name="caster"> <!-- Caster link -->
 			<visual>
-				<origin rpy="${PI/2} 0 ${PI/2}"/>
 				<geometry>
 					<cylinder length="${casterWidth}" radius="${casterRadius}"/>
@@ -12,5 +11,4 @@
 			</visual>
 			<collision>
-				<origin rpy="${PI/2} 0 ${PI/2}"/>
 				<geometry>
 					<cylinder length="${casterWidth}" radius="${casterRadius}"/>
@@ -18,7 +16,6 @@
 			</collision>
 			<inertial>
-				<origin rpy="${PI/2} 0 ${PI/2}"/>
-				<mass value="5"/>
-				<inertia ixx="0.4" ixy="0.0" ixz="0.0" iyy="0.4" iyz="0.0" izz="0.2"/>
+				<mass value="0.0625"/>
+				<inertia ixx="0.00000791" ixy="0.0" ixz="0.0" iyy="0.00000791" iyz="0.0" izz="0.00001582"/>
 			</inertial>
 		</link>
@@ -27,5 +24,5 @@
 		  <parent link="base_link"/>
 		  <child link="caster"/>
-		  <axis xyz="1 0 0"/>
+		  <axis xyz="0 0 -1"/>
 		  <insert_block name="origin"/>
 		</joint>

File: src/mag_simulation/mag_description/urdf/parts/chassis.xacro (robot description, xacro)
@@ -3,10 +3,8 @@
   <xacro:macro name="chassis" params="width length height *origin">
 		<!-- URDF description -->
-		<link name="base_footprint"> <!-- Link to apply the base_footprint to base_link TF -->
-			<origin xyz="0 0 0" rpy="0 0 0" />
-		</link>
+		<link name="base_footprint"/> <!-- Link to apply the base_footprint to base_link TF -->
 		<link name="base_link"> <!-- Main chassis link -->
 			<visual>
-				<origin xyz="0 0 ${height/2}"/>
+				<origin xyz="0 0 0"/>
 				<geometry>
 					<box size="${width} ${length} ${height}"/>
@@ -15,5 +13,5 @@
 			</visual>
 			<collision>
-				<origin xyz="0 0 ${height/2}"/>
+				<origin xyz="0 0 0"/>
 				<geometry>
 					<box size="${width} ${length} ${height}"/>
@@ -21,7 +19,7 @@
 			</collision>
 			<inertial>
-				<origin xyz="0 0 ${height/2}"/>
-				<mass value="20"/>
-				<inertia ixx="0.4" ixy="0.0" ixz="0.0" iyy="0.4" iyz="0.0" izz="0.2"/>
+				<origin xyz="0 0 0"/>
+				<mass value="2.25"/>
+				<inertia ixx="0.02860811" ixy="0.0" ixz="0.0" iyy="0.065872155" iyz="0.0" izz="0.03901133"/>
 			</inertial>
 		</link>

File: src/mag_simulation/mag_description/urdf/parts/wheel.xacro (robot description, xacro)
@@ -5,5 +5,4 @@
   	<link name="${name}"> <!-- Motorized wheel link -->
 			<visual>
-				<origin rpy="${PI/2} 0 ${PI/2}"/>
 				<geometry>
 					<cylinder length="${wheelWidth}" radius="${wheelRadius}"/>
@@ -12,5 +11,4 @@
 			</visual>
 			<collision>
-				<origin rpy="${PI/2} 0 ${PI/2}"/>
 				<geometry>
 					<cylinder length="${wheelWidth}" radius="${wheelRadius}"/>
@@ -18,7 +16,6 @@
 			</collision>
 			<inertial>
-				<origin rpy="${PI/2} 0 ${PI/2}"/>
-				<mass value="10"/>
-				<inertia ixx="0.4" ixy="0.0" ixz="0.0" iyy="0.4" iyz="0.0" izz="0.2"/>
+				<mass value="0.05"/>
+				<inertia ixx="0.000025313" ixy="0.0" ixz="0.0" iyy="0.000025313" iyz="0.0" izz="0.000050625"/>
 			</inertial>
 		</link>
@@ -27,5 +24,5 @@
 		  <parent link="base_link"/>
 		  <child link="${name}"/>
-		  <axis xyz="-1 0 0"/>
+		  <axis xyz="0 0 -1"/>
 		  <insert_block name="origin" />
 		</joint>

File: src/mag_simulation/mag_description/urdf/sensors/hokuyo_laser.gazebo.xacro (robot description, xacro)
@@ -1,6 +1,6 @@
 <?xml version="1.0"?>
 <robot xmlns:xacro="http://ros.org/wiki/xacro">
-  <xacro:macro name="hokuyo_laser_gazebo" params="topic">
-    <gazebo reference="hokuyo_link">
+  <xacro:macro name="hokuyo_laser_gazebo" params="topic laserHeight">
+    <gazebo reference="hokuyo_base">
       <sensor type="ray" name="hokuyo_laser">
         <pose>0 0 0 0 0 0</pose>
@@ -18,14 +18,15 @@
           </scan>
           <range>
-            <min>0.1</min>
-            <max>30.0</max>
+            <min>0.25</min>
+            <max>4.0</max>
             <resolution>0.01</resolution>
           </range>
+        	<noise>
+		        <type>gaussian</type>
+		        <mean>0.0</mean>
+		        <stddev>0.01</stddev>
+		      </noise>
         </ray>
         <plugin name="gazebo_ros_hokuyo_controller" filename="libgazebo_ros_laser.so">
-          <alwaysOn>true</alwaysOn>
-          <updateRate>80</updateRate>
-          <gaussianNoise>0.005</gaussianNoise>
-          <hokuyoMinIntensity>101</hokuyoMinIntensity>
           <topicName>${topic}</topicName>
           <frameName>hokuyo_link</frameName>

File: src/mag_simulation/mag_description/urdf/sensors/hokuyo_laser.xacro (robot description, xacro)
@@ -4,10 +4,13 @@
        xmlns:interface="http://playerstage.sourceforge.net/gazebo/xmlschema/#interface"
        xmlns:xacro="http://ros.org/wiki/xacro">
+  <xacro:property name="laserWidth" value="0.05"/> <!-- Width of the base -->
+  <xacro:property name="laserLength" value="0.05"/> <!-- Length of the base -->
+  <xacro:property name="laserHeight" value="0.07"/> <!-- Height -->
 	<!-- Inlude Gazebo element -->
-  <include filename="$(find mag_description)/urdf/sensors/hokuyo_laser.gazebo.xacro" />
+  <xacro:include filename="$(find mag_description)/urdf/sensors/hokuyo_laser.gazebo.xacro" />
   <xacro:macro name="hokuyo_laser" params="parent *origin topic">
-    <link name="hokuyo_link" type="laser">
+    <link name="hokuyo_base" type="laser">
 		  <visual>
-		  	<origin xyz="0 0 0.07" />
+		  	<origin xyz="0 0 0" />
 		    <geometry>
 					<mesh filename="package://mag_description/meshes/hokuyo_laser.dae"/>
@@ -15,11 +18,11 @@
 		  </visual>
 		  <collision>
-		  	<origin xyz="0 0 0.7" />
+		  	<origin xyz="0 0 0" />
 		    <geometry>
-		      <box size="0.05 0.05 0.1" />
+		      <box size="${laserWidth} ${laserLength} ${laserHeight}" />
 		    </geometry>
 		  </collision>
       <inertial>
-		  	<origin xyz="0 0 0.07" />
+		  	<origin xyz="0 0 ${laserHeight/2}" />
         <mass value="0.1" />
         <inertia ixx="0.0001" ixy="0" ixz="0" iyy="0.0001" iyz="0" izz="0.0001" />
@@ -28,10 +31,17 @@
     <joint name="hokuyo_joint" type="fixed">
       <parent link="${parent}"/>
-      <child link="hokuyo_link"/>
+      <child link="hokuyo_base"/>
       <axis xyz="0 1 0" />
       <insert_block name="origin" />
     </joint>
-    <!-- Gazebo elements -->
-    <xacro:hokuyo_laser_gazebo topic="${topic}"/>
+		<link name="hokuyo_link"/> <!-- Dummy link to correct the sensor in gazebo -->
+		<joint name="laser_joint" type="fixed">
+			<parent link="hokuyo_base"/>
+			<child link="hokuyo_link"/>
+			<axis xyz="0 1 0"/>
+			<origin xyz="0 0 ${laserHeight/2-0.005}" rpy="0 0 0"/>
+		</joint>
+	  <!-- Gazebo elements -->
+	  <xacro:hokuyo_laser_gazebo topic="${topic}" laserHeight="${laserHeight}"/>
   </xacro:macro>
 </robot>

File: src/mag_simulation/mag_description/urdf/sensors/microstrain.xacro (robot description, xacro)
@@ -4,22 +4,25 @@
 				xmlns:interface="http://playerstage.sourceforge.net/gazebo/xmlschema/#interface"
 				xmlns:xacro="http://ros.org/wiki/xacro">
+  <xacro:property name="imuWidth" value="0.0173"/> <!-- Width of the base -->
+  <xacro:property name="imuLength" value="0.01585"/> <!-- Length of the base -->
+  <xacro:property name="imuHeight" value="0.01241"/> <!-- Height -->
 	<!-- Include Gazebo element -->
-	<include filename="$(find mag_description)/urdf/sensors/microstrain.gazebo.xacro" />
+	<xacro:include filename="$(find mag_description)/urdf/sensors/microstrain.gazebo.xacro" />
 	<xacro:macro name="microstrain" params="parent *origin topic">
 		<link name="microstrain_link">
 		  <visual>
-		    <insert_block name="origin" />
+		    <origin xyz="0 0 ${imuHeight/2}"/>
 		    <geometry>
-		      <box size="0.0173 0.01585 0.01241" />
+		      <box size="${imuWidth} ${imuLength} ${imuHeight}" />
 		    </geometry>
 		  </visual>
 		  <collision>
-		    <insert_block name="origin" />
+		    <origin xyz="0 0 ${imuHeight/2}"/>
 		    <geometry>
-		      <box size="0.0173 0.01585 0.01241" />
+		      <box size="${imuWidth} ${imuLength} ${imuHeight}" />
 		    </geometry>
 		  </collision>
 			<inertial>
-		    <insert_block name="origin" />
+		    <origin xyz="0 0 ${imuHeight/2}"/>
 				<mass value="0.01" />
 				<inertia ixx="0.0001" ixy="0" ixz="0" iyy="0.0001" iyz="0" izz="0.0001" />

Commit message: Minor fixes to urdf

File: src/mag_simulation/mag_description/urdf/magabot.xacro (robot description, xacro)
@@ -12,5 +12,5 @@
   <xacro:property name="casterWidth" value="0.020"/> <!-- Width of non-motorized wheel -->
   <!-- Magabot TFs -->
-  <xacro:macro name="footprint_tf"> <origin xyz="0 0 ${height/2+0.0307}" rpy="0 0 0"/> </xacro:macro>
+  <xacro:macro name="_tf"> <origin xyz="0 0 ${height/2+0.0307}" rpy="0 0 0"/> </xacro:macro>
   <xacro:macro name="wheel_tf" params="reflect"> <origin xyz="${reflect*.1725} .0455 ${-height/2+0.0143}" rpy="${PI/2} 0 ${PI/2}"/> </xacro:macro>
   <xacro:macro name="caster_tf"> <origin xyz="0 -0.169 ${-height/2-0.0092}" rpy="${PI/2} 0 ${PI/2}"/> </xacro:macro>
@@ -34,8 +34,8 @@
   </xacro:chassis>
   <xacro:wheel name="leftwheel" wheelWidth="${wheelWidth}" wheelRadius="${wheelRadius}">
-  	<xacro:wheel_tf reflect="-1" />
+  	<xacro:wheel_tf reflect="1" />
   </xacro:wheel>
   <xacro:wheel name="rightwheel" wheelWidth="${wheelWidth}" wheelRadius="${wheelRadius}">
-  	<xacro:wheel_tf reflect="1" />
+  	<xacro:wheel_tf reflect="-1" />
   </xacro:wheel>
   <xacro:caster casterRadius="${casterRadius}" casterWidth="${casterWidth}">

Commit message: Rolled back some navigation changes and update some parameters for hydro

File: src/mag_simulation/mag_description/urdf/magabot.xacro (robot description, xacro)
@@ -12,10 +12,10 @@
   <xacro:property name="casterWidth" value="0.020"/> <!-- Width of non-motorized wheel -->
   <!-- Magabot TFs -->
-  <xacro:macro name="_tf"> <origin xyz="0 0 ${height/2+0.0307}" rpy="0 0 0"/> </xacro:macro>
+  <xacro:macro name="base_tf"> <origin xyz="0 0 ${height/2+0.0307}" rpy="0 0 0"/> </xacro:macro>
   <xacro:macro name="wheel_tf" params="reflect"> <origin xyz="${reflect*.1725} .0455 ${-height/2+0.0143}" rpy="${PI/2} 0 ${PI/2}"/> </xacro:macro>
   <xacro:macro name="caster_tf"> <origin xyz="0 -0.169 ${-height/2-0.0092}" rpy="${PI/2} 0 ${PI/2}"/> </xacro:macro>
   <!-- Sensor TFs -->
   <xacro:macro name="hokuyo_tf"> <origin xyz="0 0.0305 ${height/2+0.035}" rpy="0 0 ${PI/2}"/> </xacro:macro>
-	<xacro:macro name="wiimote_tf"> <origin xyz="0 -0.0721 ${height/2}" rpy="0 0 0"/> </xacro:macro>
+	<xacro:macro name="wiimote_tf"> <origin xyz="0 -0.0721 ${height/2}" rpy="0 0 ${PI/2}"/> </xacro:macro>
   <!-- Import Gazebo plugins -->
   <xacro:include filename="$(find mag_description)/urdf/magabot.gazebo" />
@@ -31,5 +31,5 @@
   <!-- ........... MAGABOT PARTS ........... -->
   <xacro:chassis width="${width}" length="${length}" height="${height}">
-  	<xacro:footprint_tf/>
+  	<xacro:base_tf/>
   </xacro:chassis>
   <xacro:wheel name="leftwheel" wheelWidth="${wheelWidth}" wheelRadius="${wheelRadius}">

File: src/mag_simulation/mag_description/urdf/sensors/microstrain.gazebo.xacro (robot description, xacro)
@@ -13,5 +13,5 @@
         <gaussianNoise>0.0000000289</gaussianNoise> <!-- 0.00017 * 0.00017 -->
         <xyzOffset>0 0 0</xyzOffset>
-        <rpyOffset>0 -180 0</rpyOffset>
+        <rpyOffset>0 0 0</rpyOffset>
       </plugin>
     </gazebo>

Commit message: URDF fixed and working completely, navigation somewhat tuned

File: src/mag_simulation/mag_description/urdf/magabot.xacro (robot description, xacro)
@@ -12,10 +12,10 @@
   <xacro:property name="casterWidth" value="0.020"/> <!-- Width of non-motorized wheel -->
   <!-- Magabot TFs -->
-  <xacro:macro name="base_tf"> <origin xyz="0 0 ${height/2+0.0307}" rpy="0 0 0"/> </xacro:macro>
+  <xacro:macro name="base_tf"> <origin xyz="0 0 ${height/2+0.0307}" rpy="0 0 -${PI/2}"/> </xacro:macro>
   <xacro:macro name="wheel_tf" params="reflect"> <origin xyz="${reflect*.1725} .0455 ${-height/2+0.0143}" rpy="${PI/2} 0 ${PI/2}"/> </xacro:macro>
   <xacro:macro name="caster_tf"> <origin xyz="0 -0.169 ${-height/2-0.0092}" rpy="${PI/2} 0 ${PI/2}"/> </xacro:macro>
   <!-- Sensor TFs -->
-  <xacro:macro name="hokuyo_tf"> <origin xyz="0 0.0305 ${height/2+0.035}" rpy="0 0 ${PI/2}"/> </xacro:macro>
-	<xacro:macro name="wiimote_tf"> <origin xyz="0 -0.0721 ${height/2}" rpy="0 0 ${PI/2}"/> </xacro:macro>
+  <xacro:macro name="hokuyo_tf"> <origin xyz="0 0.0305 ${height/2+0.07}" rpy="0 0 ${PI/2}"/> </xacro:macro>
+	<xacro:macro name="wiimote_tf"> <origin xyz="0 -0.0721 ${height/2}" rpy="0 0 0"/> </xacro:macro>
   <!-- Import Gazebo plugins -->
   <xacro:include filename="$(find mag_description)/urdf/magabot.gazebo" />

File: src/mag_simulation/mag_description/urdf/sensors/hokuyo_laser.xacro (robot description, xacro)
@@ -12,5 +12,5 @@
     <link name="hokuyo_base" type="laser">
 		  <visual>
-		  	<origin xyz="0 0 0" />
+		  	<origin xyz="0 0 -${laserHeight/2}" />
 		    <geometry>
 					<mesh filename="package://mag_description/meshes/hokuyo_laser.dae"/>
@@ -18,5 +18,5 @@
 		  </visual>
 		  <collision>
-		  	<origin xyz="0 0 0" />
+		  	<origin xyz="0 0 -${laserHeight/2}" />
 		    <geometry>
 		      <box size="${laserWidth} ${laserLength} ${laserHeight}" />
@@ -24,5 +24,5 @@
 		  </collision>
       <inertial>
-		  	<origin xyz="0 0 ${laserHeight/2}" />
+		  	<origin xyz="0 0 -${laserHeight/4}" />
         <mass value="0.1" />
         <inertia ixx="0.0001" ixy="0" ixz="0" iyy="0.0001" iyz="0" izz="0.0001" />

File: src/mag_simulation/mag_description/urdf/sensors/microstrain.gazebo.xacro (robot description, xacro)
@@ -3,4 +3,5 @@
        xmlns:interface="http://playerstage.sourceforge.net/gazebo/xmlschema/#interface"
        xmlns:xacro="http://ros.org/wiki/xacro">
+  <xacro:property name="PI" value="3.14159"/>
   <xacro:macro name="microstrain_gazebo" params="topic">
     <gazebo>

File: src/mag_simulation/mag_description/urdf/sensors/microstrain.xacro (robot description, xacro)
@@ -4,6 +4,8 @@
 				xmlns:interface="http://playerstage.sourceforge.net/gazebo/xmlschema/#interface"
 				xmlns:xacro="http://ros.org/wiki/xacro">
-  <xacro:property name="imuWidth" value="0.0173"/> <!-- Width of the base -->
-  <xacro:property name="imuLength" value="0.01585"/> <!-- Length of the base -->
+ <!-- <xacro:property name="imuWidth" value="0.0173"/> --> <!-- Width of the base -->
+ <!-- <xacro:property name="imuLength" value="0.01585"/> --> <!-- Length of the base -->
+  <xacro:property name="imuWidth" value="0.05"/> <!-- Width of the base -->
+  <xacro:property name="imuLength" value="0.15"/> <!-- Length of the base -->
   <xacro:property name="imuHeight" value="0.01241"/> <!-- Height -->
 	<!-- Include Gazebo element -->
