Commit message: Made some alterations to magabot and imu pacakages

File: src/mag_description/urdf/parts/wheel.xacro (robot description, xacro)
@@ -17,5 +17,5 @@
 			<inertial>
 				<mass value="0.05"/>
-				<inertia ixx="0.000025313" ixy="0.0" ixz="0.0" iyy="0.000025313" iyz="0.0" izz="0.000050625"/>
+				<inertia ixx="0.025313" ixy="0.0" ixz="0.0" iyy="0.025313" iyz="0.0" izz="0.050625"/>
 			</inertial>
 		</link>
