Commit message: Fixed magabot launchers for udev

File: src/mag_description/urdf/magabot.xacro (robot description, xacro)
@@ -17,5 +17,5 @@
   <!-- Sensor TFs -->
   <xacro:macro name="hokuyo_tf"> <origin xyz="0 0.0305 ${height/2+0.07}" rpy="0 0 ${PI/2}"/> </xacro:macro>
-	<xacro:macro name="wiimote_tf"> <origin xyz="0 -0.0721 ${height/2}" rpy="0 0 0"/> </xacro:macro>
+	<xacro:macro name="imu_tf"> <origin xyz="0 -0.0721 ${height/2}" rpy="0 0 0"/> </xacro:macro>
   <!-- Import Gazebo plugins -->
   <xacro:include filename="$(find mag_description)/urdf/magabot.gazebo" />
@@ -26,5 +26,5 @@
   <!-- Import Sensors -->
   <xacro:include filename="$(find mag_description)/urdf/sensors/hokuyo_laser.xacro" />
-  <xacro:include filename="$(find mag_description)/urdf/sensors/microstrain.xacro" />
+  <xacro:include filename="$(find mag_description)/urdf/sensors/imu.xacro" />
   <!-- Import Materials -->
   <xacro:include filename="$(find mag_description)/urdf/materials/materials.xacro" />
@@ -46,7 +46,7 @@
   	<xacro:hokuyo_tf/>
   </xacro:hokuyo_laser>
-  <xacro:microstrain parent="base_link" topic="imu_data">
-  	<xacro:wiimote_tf/>
-  </xacro:microstrain>
+  <xacro:imu parent="base_link" link="imu" topic="imu_data">
+  	<xacro:imu_tf/>
+  </xacro:imu>
   <!-- ....... GAZEBO PLUGINS ....... -->
   <xacro:plugins_gazebo topic="odom_combined" wheelSep="${wheelSep}" wheelRad="${wheelRadius}"/>

File: src/mag_description/urdf/sensors/imu.gazebo.xacro (robot description, xacro)
@@ -4,10 +4,10 @@
        xmlns:xacro="http://ros.org/wiki/xacro">
   <xacro:property name="PI" value="3.14159"/>
-  <xacro:macro name="microstrain_gazebo" params="topic">
+  <xacro:macro name="imu_gazebo" params="topic link">
     <gazebo>
       <plugin name="imu_controller" filename="libgazebo_ros_imu.so">
         <alwaysOn>true</alwaysOn>
         <updateRate>80</updateRate>
-        <bodyName>microstrain_link</bodyName>
+        <bodyName>${link}</bodyName>
         <topicName>${topic}</topicName>
         <serviceName>/default_imu</serviceName>

File: src/mag_description/urdf/sensors/imu.xacro (robot description, xacro)
@@ -10,7 +10,7 @@
   <xacro:property name="imuHeight" value="0.01241"/> <!-- Height -->
 	<!-- Include Gazebo element -->
-	<xacro:include filename="$(find mag_description)/urdf/sensors/microstrain.gazebo.xacro" />
-	<xacro:macro name="microstrain" params="parent *origin topic">
-		<link name="microstrain_link">
+	<xacro:include filename="$(find mag_description)/urdf/sensors/imu.gazebo.xacro" />
+	<xacro:macro name="imu" params="parent link *origin topic">
+		<link name="${link}">
 		  <visual>
 		    <origin xyz="0 0 ${imuHeight/2}"/>
@@ -31,12 +31,12 @@
 			</inertial>
 		</link>
-		<joint name="microstrain_joint" type="fixed">
+		<joint name="imu_joint" type="fixed">
 			<axis xyz="0 1 0" />
 			<insert_block name="origin" />
 			<parent link="${parent}"/>
-			<child link="microstrain_link"/>
+			<child link="${link}"/>
 		</joint>
 		<!-- Gazebo element -->
-		<xacro:microstrain_gazebo topic="${topic}"/>
+		<xacro:imu_gazebo topic="${topic}" link="${link}"/>
 	</xacro:macro>
 </robot>
